Commit message: camera pointclouds works only for ignition gazebo version

File: robot_description/urdf/donkey_sensors.urdf (robot description, URDF)
Before this commit: robot ackmann_robot, 8 links, 7 joints
Links:
- added link ${l515_name}_depth_frame
- added link ${l515_name}_depth_optical_frame
- added link ${l515_name}_link; collision box size=0.012 0.132 0.020; visual box size=0.012 0.132 0.020
Joints:
- added joint ${l515_name}_depth_joint: type fixed, parent ${l515_name}_link, child ${l515_name}_depth_frame, origin xyz=0.005 0.028 0.013 rpy=0 0 0
- added joint ${l515_name}_depth_optical_joint: type fixed, parent ${l515_name}_depth_frame, child ${l515_name}_depth_optical_frame, origin xyz=0 0 0 rpy=${PI/2} 0 ${-PI/2}
- added joint ${l515_name}_joint: type fixed, parent $(arg ns)/base_link, child ${l515_name}_link, origin xyz=0.1 0 0.07 rpy=0 0 0

Commit message: rtabmap works

File: robot_description/urdf/donkey_sensors.urdf (robot description, URDF)
Before this commit: robot ackmann, 11 links, 10 joints
Joints:
- joint ${l515_name}_depth_optical_joint: origin xyz=0 0 0 rpy=${PI/2} 0 ${-PI/2} -> xyz=0 0 0 rpy=${-PI/2} 0 ${-PI/2}

Commit message: rgbd topic stopped publishing

File: robot_description/urdf/donkey_sensors.urdf (robot description, URDF)
Before this commit: robot ackmann, 11 links, 10 joints
Links:
- removed link ${l515_name}_depth_frame
- removed link ${l515_name}_depth_optical_frame
- removed link ${l515_name}_link
Joints:
- removed joint ${l515_name}_depth_joint
- removed joint ${l515_name}_depth_optical_joint
- removed joint ${l515_name}_joint

File: robot_description/urdf/realsense/_l515.urdf.xacro (robot description, xacro)
@@ -81,6 +81,4 @@
       </collision>
       <inertial>
-        <!-- The following are not reliable values, and should not be used for modeling -->
-        <!-- calculated assuming full cylinder as described here: https://en.wikipedia.org/wiki/List_of_moments_of_inertia -->
         <mass value="0.095" />
         <origin xyz="0 0 0" />
