Commit message: add imu sensor

File: robot_description/urdf/realsense/_l515.urdf.xacro (robot description, xacro)
@@ -144,4 +144,5 @@
       <link name="${name}_accel_frame" />
       <link name="${name}_accel_optical_frame" />
+      <link name="${name}_imu_optical_frame" />
       <joint name="${name}_gyro_joint" type="fixed">
         <origin xyz = "${l515_cam_color_to_imu_px} ${l515_cam_color_to_imu_py} ${l515_cam_color_to_imu_pz}" rpy = "${l515_cam_color_to_imu_rx} ${l515_cam_color_to_imu_ry} ${l515_cam_color_to_imu_rz}" />
@@ -164,4 +165,9 @@
         <child link="${name}_accel_optical_frame" />
       </joint>
+      <joint name="${name}_imu_optical_joint" type="fixed">
+        <origin xyz = "${l515_cam_color_to_imu_px} ${l515_cam_color_to_imu_py} ${l515_cam_color_to_imu_pz}" rpy = "${-M_PI/2} 0 ${-M_PI/2}" />
+        <parent link="${name}_link" />
+        <child link="${name}_imu_optical_frame" />
+      </joint>
     </xacro:if>
     <xacro:if value="${add_plug}">

Commit message: VIO works for only odom launch, to be integrated with slam launch

File: robot_description/urdf/realsense/_l515.urdf.xacro (robot description, xacro)
@@ -167,4 +167,5 @@
       <joint name="${name}_imu_optical_joint" type="fixed">
         <origin xyz = "${l515_cam_color_to_imu_px} ${l515_cam_color_to_imu_py} ${l515_cam_color_to_imu_pz}" rpy = "${-M_PI/2} 0 ${-M_PI/2}" />
+        <!-- <origin xyz = "${l515_cam_color_to_imu_px} ${l515_cam_color_to_imu_py} ${l515_cam_color_to_imu_pz}" rpy = "0 0 0" /> -->
         <parent link="${name}_link" />
         <child link="${name}_imu_optical_frame" />
