Commit message: preparing ekf fusion of imu and VO

File: robot_description/urdf/realsense/_d435i_imu_modules.urdf.xacro (robot description, xacro)
@@ -14,4 +14,5 @@
       <link name="${name}_gyro_frame" />
       <link name="${name}_gyro_optical_frame" />
+      <link name="${name}_imu_optical_frame" />
       <joint name="${name}_accel_joint" type="fixed">
         <origin xyz = "-0.01174 -0.00552 0.0051" rpy = "0 0 0" />
@@ -34,4 +35,8 @@
         <child link="${name}_gyro_optical_frame" />
       </joint>
+      <joint name="${name}_imu_optical_joint" type="fixed">
+        <origin xyz = "-0.01174 -0.00552 0.0051" rpy = "${-M_PI/2} 0 ${-M_PI/2}" />
+        <parent link="${name}_link" />
+        <child link="${name}_imu_optical_frame" />
     </xacro:if>
   </xacro:macro>

Commit message: joint_state is not published

File: robot_description/urdf/realsense/_d435i_imu_modules.urdf.xacro (robot description, xacro)
@@ -14,4 +14,5 @@
       <link name="${name}_gyro_frame" />
       <link name="${name}_gyro_optical_frame" />
+      <link name="${name}_imu_frame" />
       <link name="${name}_imu_optical_frame" />
       <joint name="${name}_accel_joint" type="fixed">
@@ -35,8 +36,14 @@
         <child link="${name}_gyro_optical_frame" />
       </joint>
+      <joint name="${name}_imu_joint" type="fixed">
+        <origin xyz = "0 0 0" rpy = "0 0 0" />
+        <parent link="${name}_gyro_frame" />
+        <child link="${name}_imu_frame" />
+      </joint>
       <joint name="${name}_imu_optical_joint" type="fixed">
-        <origin xyz = "-0.01174 -0.00552 0.0051" rpy = "${-M_PI/2} 0 ${-M_PI/2}" />
-        <parent link="${name}_link" />
+        <origin xyz = "0 0 0" rpy = "${-M_PI/2} 0 ${-M_PI/2}" />
+        <parent link="${name}_imu_frame" />
         <child link="${name}_imu_optical_frame" />
+      </joint>
     </xacro:if>
   </xacro:macro>
