Commit message: put sensor plugin into urdf file

File: robot_description/urdf/realsense/_d435i.urdf.xacro (robot description, xacro)
@@ -9,9 +9,13 @@
   <xacro:include filename="$(find realsense2_description)/urdf/_d435.urdf.xacro"/>
   <xacro:include filename="$(find robot_description)/urdf/realsense/_d435i_imu_modules.urdf.xacro"/>
-  <xacro:macro name="sensor_d435i" params="parent *origin name:=camera use_nominal_extrinsics:=false">
+  <xacro:include filename="$(find robot_description)/urdf/realsense/_d435i_sensors.urdf.xacro"/>
+  <xacro:macro name="sensor_d435i" params="parent *origin name:=camera use_nominal_extrinsics:=false add_plug:=false use_mesh:=true add_sensors:=true">
     <xacro:sensor_d435 parent="${parent}" name="${name}" use_nominal_extrinsics="${use_nominal_extrinsics}">
       <xacro:insert_block name="origin" />
     </xacro:sensor_d435>
     <xacro:d435i_imu_modules name="${name}" use_nominal_extrinsics="${use_nominal_extrinsics}"/>
+    <xacro:if value="${add_sensors}">
+      <xacro:gazebo_d435i parent="${parent}" name="${name}" width="640" height="480" fov="1.39626" image_fps="30" accel_fps="62.5" gyro_fps="200"/>
+    </xacro:if>
   </xacro:macro>
 </robot>

File: robot_description/urdf/realsense/_l515.urdf.xacro (robot description, xacro)
@@ -10,5 +10,6 @@
   <xacro:include filename="$(find realsense2_description)/urdf/_materials.urdf.xacro" />
   <xacro:include filename="$(find realsense2_description)/urdf/_usb_plug.urdf.xacro" /> <!-- this specific plug does not apply to L515 -->
-  <xacro:macro name="sensor_l515" params="parent *origin name:=camera use_nominal_extrinsics:=false add_plug:=false use_mesh:=true">
+  <xacro:include filename="$(find robot_description)/urdf/realsense/_l515_sensors.urdf.xacro"/>
+  <xacro:macro name="sensor_l515" params="parent *origin name:=camera use_nominal_extrinsics:=false add_plug:=false use_mesh:=true add_sensors:=true">
     <xacro:property name="M_PI" value="3.1415926535897931" />
     <!-- The following values are approximate, and the camera node
@@ -177,4 +178,7 @@
       </xacro:usb_plug>
     </xacro:if>
+    <xacro:if value="${add_sensors}">
+      <xacro:gazebo_l515 parent="${parent}" name="${name}" width="640" height="480" fov="1.39626" image_fps="30" accel_fps="62.5" gyro_fps="200"/>
+    </xacro:if>
   </xacro:macro>
 </robot>

File: robot_description/urdf/realsense/_t265_sensors.urdf.xacro (robot description, xacro)
@@ -5,5 +5,5 @@
                                           fisheye_width:=848
                                           fisheye_height:=800
-                                          fov:=3.5
+                                          fov:=2.9
                                           fisheye_fps:=30
                                           accel_fps:=62.5
@@ -31,5 +31,9 @@
           </clip>
         <lens>
-          <intrinsics>
+          <type>equisolid_angle</type>
+          <scale_to_hfov>true</scale_to_hfov>
+          <cutoff_angle>${fov/2}</cutoff_angle>  <!-- 85° cutoff -->
+          <env_texture_size>1024</env_texture_size>
+          <!-- <intrinsics>
             <fx>${fisheye_width / (2 * tan(fov/2))}</fx>
             <fy>${fisheye_width / (2 * tan(fov/2))}</fy>
@@ -43,4 +47,13 @@
             <p_cy>${fisheye_height / 2}</p_cy>
           </projection>
+          <distortion>
+            <k1>-0.15</k1>
+            <k2>0.041209</k2>
+            <k3>-0.037267</k3>
+            <k4>0.007446</k4>
+            <p1>0</p1>
+            <p2>0</p2>
+            <center>0.5 0.5</center>
+          </distortion> -->
         </lens>
         </camera>
@@ -64,5 +77,9 @@
           </clip>
         <lens>
-          <intrinsics>
+          <type>equisolid_angle</type>
+          <scale_to_hfov>true</scale_to_hfov>
+          <cutoff_angle>${fov/2}</cutoff_angle>  <!-- 85° cutoff -->
+          <env_texture_size>1024</env_texture_size>
+          <!-- <intrinsics>
             <fx>${fisheye_width / (2 * tan(fov/2))}</fx>
             <fy>${fisheye_width / (2 * tan(fov/2))}</fy>
@@ -75,5 +92,5 @@
             <p_cx>${fisheye_width / 2}</p_cx>
             <p_cy>${fisheye_height / 2}</p_cy>
-          </projection>
+          </projection> -->
         </lens>
         </camera>
