Commit message: odom fusion only works with simulation

File: robot_description/urdf/realsense/_l515_sensors.urdf.xacro (robot description, xacro)
@@ -30,8 +30,29 @@
           </clip>
           <lens>
-            <type>stereographic</type>
+            <type>pinhole</type>
             <scale_to_hfov>true</scale_to_hfov>
-            <cutoff_angle>${fov/2}</cutoff_angle>  <!-- 85° cutoff -->
+            <cutoff_angle>${fov/2}</cutoff_angle>
             <env_texture_size>1024</env_texture_size>
+            <intrinsics>
+              <fx>${width / (2 * tan(fov/2))}</fx>
+              <fy>${width / (2 * tan(fov/2))}</fy>
+              <cx>${width / 2}</cx>
+              <cy>${height / 2}</cy>
+            </intrinsics>
+            <projection>
+              <p_fx>${width / (2 * tan(fov/2))}</p_fx>
+              <p_fy>${width / (2 * tan(fov/2))}</p_fy>
+              <p_cx>${width / 2}</p_cx>
+              <p_cy>${height / 2}</p_cy>
+            </projection>
+            <!-- <distortion>
+              <k1>-0.15</k1>
+              <k2>0.041209</k2>
+              <k3>-0.037267</k3>
+              <k4>0.007446</k4>
+              <p1>0</p1>
+              <p2>0</p2>
+              <center>0.5 0.5</center>
+            </distortion> -->
           </lens>
           <optical_frame_id>${name}_depth_optical_frame</optical_frame_id>

File: robot_description/urdf/realsense/_t265.urdf.xacro (robot description, xacro)
@@ -20,8 +20,16 @@
       <color rgba="0.5 0.5 0.5 1"/>
     </material>
+    <!-- camera body, with origin at camera_link -->
+    <joint name="${name}_link_joint" type="fixed">
+      <!-- <origin xyz="0 0 0" rpy="0 0 0"/> -->
+      <xacro:insert_block name="origin"/>
+      <parent link="${parent}"/>
+      <child link="${name}_link"/>
+    </joint>
+    <link name="${name}_link"/>
     <!-- camera body, with origin at camera_pose_frame -->
     <joint name="${name}_pose_joint" type="fixed">
       <xacro:insert_block name="origin"/>
-      <parent link="${parent}"/>
+      <parent link="${name}_link"/>
       <child link="${name}_pose_frame"/>
     </joint>
@@ -47,11 +55,4 @@
       </inertial>
     </link>
-    <!-- camera body, with origin at camera_link -->
-    <joint name="${name}_link_joint" type="fixed">
-      <origin xyz="0 0 0" rpy="0 0 0"/>
-      <parent link="${name}_pose_frame"/>
-      <child link="${name}_link"/>
-    </joint>
-    <link name="${name}_link"/>
     <joint name="${name}_fisheye1_joint" type="fixed">
       <origin xyz="${fisheye1_offset_x} ${fisheye1_offset_y} ${fisheye1_offset_z}" rpy="${-M_PI} 0 ${-M_PI}"/>

File: robot_description/urdf/realsense/_t265_sensors.urdf.xacro (robot description, xacro)
@@ -125,5 +125,5 @@
         <dimensions>3</dimensions>
         <odom_frame>odom_frame</odom_frame>
-        <robot_base_frame>${name}/pose_frame</robot_base_frame>
+        <robot_base_frame>${name}_pose_frame</robot_base_frame>
         <publish_link_pose>true</publish_link_pose>
         <tf_topic>$(arg ns)/tf</tf_topic>
